Commit message: edited urdf

File: xarm_description/urdf/lite6/lite6.urdf.xacro (robot description, xacro)
@@ -24,4 +24,25 @@
       <xacro:property name="inertial_params" value="${load_yaml(link_inertial_params_file)}"/>
     </xacro:unless>
+    <!---->
+  <link name="box">
+    <visual>
+      <origin xyz="0 0 0.5" rpy="0 0 0"/>
+      <geometry>
+        <box size="1 1 1"/>
+      </geometry>
+    </visual>
+    <collision>
+      <origin xyz="0 0 0.5" rpy="0 0 0"/>
+      <geometry>
+        <box size="1 1 1"/>
+      </geometry>
+    </collision>
+  </link>
+    <joint name="box_joint" type="fixed">
+      <origin xyz="0 0 1" rpy="0 0 0" />
+      <parent link="box" />
+      <child link="link_base" />
+    </joint>
+    <!---->
     <link name="${prefix}link_base">
       <inertial>

File: xarm_description/urdf/xarm_device_macro.xacro (robot description, xacro)
@@ -64,5 +64,5 @@
     <joint name="${prefix}world_joint" type="fixed">
       <parent link="${attach_to}" />
-      <child link = "${prefix}link_base" />
+      <child link = "box" />
       <origin xyz="${attach_xyz}" rpy="${attach_rpy}" />
     </joint>

Commit message: chnaged box position to bottom

File: xarm_description/urdf/lite6/lite6.urdf.xacro (robot description, xacro)
@@ -27,5 +27,5 @@
   <link name="box">
     <visual>
-      <origin xyz="0 0 0.5" rpy="0 0 0"/>
+      <origin xyz="0 0 -0.5" rpy="0 0 0"/>
       <geometry>
         <box size="1 1 1"/>
@@ -33,5 +33,5 @@
     </visual>
     <collision>
-      <origin xyz="0 0 0.5" rpy="0 0 0"/>
+      <origin xyz="0 0 -0.5" rpy="0 0 0"/>
       <geometry>
         <box size="1 1 1"/>
@@ -40,5 +40,5 @@
   </link>
     <joint name="box_joint" type="fixed">
-      <origin xyz="0 0 1" rpy="0 0 0" />
+      <origin xyz="0 0 0" rpy="0 0 0" />
       <parent link="box" />
       <child link="link_base" />

Commit message: edited urdf to have accurate robot hull

File: xarm_description/urdf/lite6/lite6.urdf.xacro (robot description, xacro)
@@ -27,13 +27,13 @@
   <link name="box">
     <visual>
-      <origin xyz="0 0 -0.5" rpy="0 0 0"/>
+      <origin xyz="0 0 -0.115" rpy="0 0 0"/>
       <geometry>
-        <box size="1 1 1"/>
+        <box size="0.47 0.34 0.23"/>
       </geometry>
     </visual>
     <collision>
-      <origin xyz="0 0 -0.5" rpy="0 0 0"/>
+      <origin xyz="0 0 -0.115" rpy="0 0 0"/>
       <geometry>
-        <box size="1 1 1"/>
+        <box size="0.47 0.34 0.23"/>
       </geometry>
     </collision>
